File: SSCI_SPI_LCD.sch (EAGLE design)
At the start: 5 parts

Commit message: r0.1 prototype
Parts:
- added C1, C2: (no value), mylib:C_SMD_10U_1608
- added C3, C4, C5, C6, C7, C8: (no value), mylib:C_SMD_0.1U_1005
- added GIT1: (no value), git-revision:GIT-REVISION
- added IC1: (no value), mylib:LDO4_3.3_SC82−AB
- added IC2: (no value), mylib:74LVC1G00_DRL
- added IC3: 74LVC541_RGY, mylib:74LVC541_RGY
- added IC4: (no value), mylib:IC_MEMORY_8P_23K256-I_SOP
- added IC5: (no value), mylib:74LVC1G125_DRL
- added ICON1: r0.1, mylib:ICON_REVISION_2.0
- added R1, R2, R3, R4, R5, R6: (no value), mylib:R_US_10K_1005
- added X1, X2: TSW-108-02-S-S, con-samtec.local:TSW-108-02-S-S
Connections:
- new net !CSR!: IC3.A1, R2.2, X1-4.1, X2-4.1
- new net !CSR!-: IC2.1A, IC3.Y1, IC4.!CS
- new net 3.3V: C2.1, C3.1, C4.1, C5.1, C6.1, C7.1, C8.1, IC1.OUT, IC2.VCC, IC3.VCC, IC4.!HOLD, IC4.!WP, IC4.VCC, IC5.VCC, LCD1.AVDD, LCD1.DVDD, R2.1
- new net 5V: C1.1, IC1.IN, IC1.OUT/EN/NC, X1-1.1, X2-1.1
- new net CSL: IC3.A5, R4.2, X1-7.1, X2-7.1
- new net CSL-: IC2.1B, IC3.Y5, LCD1.CS
- new net DISP: IC3.A4, R3.2, X1-6.1, X2-6.1
- new net DISP-: IC3.Y4, LCD1.DISP
- new net GND: C1.2, C2.2, C3.2, C4.2, C5.2, C6.2, C7.2, C8.2, IC1.ADJ, IC2.GND, IC3.A2, IC3.A3, IC3.G1, IC3.G2, IC3.GND, IC4.GND, IC5.GND, LCD1.GND, LCD1.GND@1, LCD1.GND@2, R1.1, R3.1, R4.1, R5.1, R6.1, X1-2.1, X2-2.1
- new net MISO: IC3.Y6, X1-5.1, X2-5.1
- new net MISO-: IC3.A6, IC4.SO, IC5.Y, LCD1.MOSI, R5.2
- new net MOSI: IC3.A0, R1.2, X1-3.1, X2-3.1
- new net MOSI-: IC3.Y0, IC4.SI, IC5.A
- new net N$2: IC2.1Y, IC5.!OE!
- new net SCK: IC3.A7, R6.2, X1-8.1, X2-8.1
- new net SCK-: IC3.Y7, IC4.SCK, LCD1.SCK

Commit message: connectors silk
Parts:
- GIT1: value (none) -> a88ec19
Changed lines of the file:
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@@
 <part name="P3" library="mylib" deviceset="PCB_CORNER" device=""/>
 <part name="P4" library="mylib" deviceset="PCB_CORNER" device=""/>
-<part name="GIT1" library="git-revision" deviceset="GIT-REVISION" device=""/>
+<part name="GIT1" library="git-revision" deviceset="GIT-REVISION" device="" value="a88ec19"/>
 <part name="FRAME1" library="frames" deviceset="A4L-LOC" device=""/>
 <part name="ICON1" library="mylib" deviceset="ICON_REVISION" device="_2.0" value="r0.1"/>

Commit message: revision 0.1
Parts:
- added ICON2: (no value), mylib:ICON_OSHW
- GIT1: value a88ec19 -> 11642e8
Connections:
- net GND: now also LCD1.PAD, LCD1.PAD@1
Other:
- moved on the sheet: C3, C5, C6, C7, C8, IC2, IC4, IC5
